File: Hardware/Sequencer/Sequencer.kicad_pcb (KiCad board)
At the start: 4 copper layers, 200 x 150 mm, 142 parts, among them J301 Conn_ST_STDC14, J601 USB_C_Receptacle_USB2.0_16P, SW301 SW_Push, SW401 SW_SP4T_NR01104, SW402 SW_SP4T_NR01104, SW403 SW_SP4T_NR01104, U1 PCA9635, U2 PCA9635, U301 STM32G474RETx, U4 MCP23017_SP, U401 MCP23017_SP, U402 MCP23017_SP, U601 USBLC6-2SC6, U602 AZ1117-3.3TRG1

Commit message: update pcb
Parts:
- removed C1, C10, C11, C12, C13, C14, C15, C16, C17, C2, C3, C4, C5, C6, C7, C8, C9: 100n, Capacitor_SMD:C_0402_1005Metric
- removed R1, R10, R12, R13, R15, R16, R18, R19, R21, R22, R24, R25, R27, R28, R3, R30, R31, R33, R34, R36, R37, R39, R4, R40, R42, R43, R45, R46, R48, R6, R7, R9: 10k, Resistor_SMD:R_0402_1005Metric
- removed U4: MCP23017_SP, Package_SO:SOIC-28W_7.5x17.9mm_P1.27mm
- added C101: 10n, Capacitor_SMD:C_0402_1005Metric, F.Cu at (83.4, 73.0)
- added C303: 10n, Capacitor_SMD:C_0402_1005Metric, F.Cu at (67.6, 97.2)
- added C308: 10n, Capacitor_SMD:C_0402_1005Metric, F.Cu at (67.6, 99.2)
- added C404: 10n, Capacitor_SMD:C_0402_1005Metric, F.Cu at (54.0, 79.5)
- added C405: 10n, Capacitor_SMD:C_0402_1005Metric, F.Cu at (56.8, 73.6)
- added C406: 10n, Capacitor_SMD:C_0402_1005Metric, F.Cu at (56.8, 75.6)
- added C407: 10n, Capacitor_SMD:C_0402_1005Metric, F.Cu at (56.8, 77.6)
- added C408: 10n, Capacitor_SMD:C_0402_1005Metric, F.Cu at (248.8, 141.5)
- added C409: 10n, Capacitor_SMD:C_0402_1005Metric, F.Cu at (59.7, 73.6)
- added C410: 10n, Capacitor_SMD:C_0402_1005Metric, F.Cu at (59.7, 75.6)
- added C411: 10n, Capacitor_SMD:C_0402_1005Metric, F.Cu at (59.7, 77.6)
- added C412: 10n, Capacitor_SMD:C_0402_1005Metric, F.Cu at (59.7, 79.5)
- added C413: 10n, Capacitor_SMD:C_0402_1005Metric, F.Cu at (62.6, 73.6)
- added C414: 10n, Capacitor_SMD:C_0402_1005Metric, F.Cu at (62.6, 75.6)
- added C415: 10n, Capacitor_SMD:C_0402_1005Metric, F.Cu at (62.6, 77.6)
- added C416: 10n, Capacitor_SMD:C_0402_1005Metric, F.Cu at (62.6, 79.5)
- added D301: LED, LED_SMD:LED_0603_1608Metric, F.Cu at (79.2, 94.3)
- added D302: LED, LED_SMD:LED_0603_1608Metric, F.Cu at (79.2, 96.9)
- added D303: LED, LED_SMD:LED_0603_1608Metric, F.Cu at (79.2, 99.5)
- added J101: LINEOUT, Connector_Audio:Jack_3.5mm_PJ320D_Horizontal, F.Cu at (75.4, 73.5)
- added R101: 10k, Resistor_SMD:R_0402_1005Metric, F.Cu at (83.5, 69.0)
- added R102: 10k, Resistor_SMD:R_0402_1005Metric, F.Cu at (83.5, 71.0)
- added R301: 10k, Resistor_SMD:R_0402_1005Metric, F.Cu at (78.7, 82.0)
- added R302: 10k, Resistor_SMD:R_0402_1005Metric, F.Cu at (78.7, 84.0)
- added R303: R_Small, Resistor_SMD:R_0402_1005Metric, F.Cu at (78.7, 86.0)
- added R304: 10k, Resistor_SMD:R_0402_1005Metric, F.Cu at (78.7, 88.0)
- added R305: 10k, Resistor_SMD:R_0402_1005Metric, F.Cu at (78.7, 90.0)
- added R306: 470, Resistor_SMD:R_0402_1005Metric, F.Cu at (78.7, 92.0)
- added R307: 10k, Resistor_SMD:R_0402_1005Metric, F.Cu at (81.6, 82.0)
- added R308: 470, Resistor_SMD:R_0402_1005Metric, F.Cu at (81.6, 84.0)
- added R309: 470, Resistor_SMD:R_0402_1005Metric, F.Cu at (81.6, 86.0)
- added R310: 10k, Resistor_SMD:R_0402_1005Metric, F.Cu at (81.6, 88.0)
- added R311: 10k, Resistor_SMD:R_0402_1005Metric, F.Cu at (81.6, 90.0)
- added R401: 0, Resistor_SMD:R_0402_1005Metric, F.Cu at (54.0, 55.7)
- added R402: 0, Resistor_SMD:R_0402_1005Metric, F.Cu at (54.0, 57.7)
- added R403: 10k, Resistor_SMD:R_0402_1005Metric, F.Cu at (54.0, 59.7)
- added R404: 10k, Resistor_SMD:R_0402_1005Metric, F.Cu at (54.0, 61.7)
- added R405: 10k, Resistor_SMD:R_0402_1005Metric, F.Cu at (54.0, 63.7)
- added R406: 10k, Resistor_SMD:R_0402_1005Metric, F.Cu at (54.0, 65.7)
- added R407: 10k, Resistor_SMD:R_0402_1005Metric, F.Cu at (54.0, 67.7)
- added R408: 10k, Resistor_SMD:R_0402_1005Metric, F.Cu at (54.0, 69.7)
- added R409: 10k, Resistor_SMD:R_0402_1005Metric, F.Cu at (54.0, 71.7)
- added R410: 10k, Resistor_SMD:R_0402_1005Metric, F.Cu at (56.9, 55.7)
- added R411: 10k, Resistor_SMD:R_0402_1005Metric, F.Cu at (65.0, 136.7)
- added R412: 10k, Resistor_SMD:R_0402_1005Metric, F.Cu at (65.0, 138.7)
- added R413: 10k, Resistor_SMD:R_0402_1005Metric, F.Cu at (65.0, 140.7)
- added R414: 10k, Resistor_SMD:R_0402_1005Metric, F.Cu at (65.0, 142.6)
- added R415: 10k, Resistor_SMD:R_0402_1005Metric, F.Cu at (65.0, 144.6)
- added R416: 10k, Resistor_SMD:R_0402_1005Metric, F.Cu at (65.0, 146.6)
- added R417: 10k, Resistor_SMD:R_0402_1005Metric, F.Cu at (65.0, 148.6)
- added R418: 10k, Resistor_SMD:R_0402_1005Metric, F.Cu at (65.0, 150.6)
- added R419: 10k, Resistor_SMD:R_0402_1005Metric, F.Cu at (56.9, 57.7)
- added R420: 10k, Resistor_SMD:R_0402_1005Metric, F.Cu at (56.9, 59.7)
- added R421: 10k, Resistor_SMD:R_0402_1005Metric, F.Cu at (56.9, 61.7)
- added R422: 10k, Resistor_SMD:R_0402_1005Metric, F.Cu at (250.7, 141.5)
- added R423: 10k, Resistor_SMD:R_0402_1005Metric, F.Cu at (56.9, 65.7)
- added R424: 10k, Resistor_SMD:R_0402_1005Metric, F.Cu at (56.9, 67.7)
- added R425: 10k, Resistor_SMD:R_0402_1005Metric, F.Cu at (56.9, 69.7)
- added R426: 10k, Resistor_SMD:R_0402_1005Metric, F.Cu at (252.6, 141.5)
- added R427: 10k, Resistor_SMD:R_0402_1005Metric, F.Cu at (67.9, 136.7)
- added R428: 10k, Resistor_SMD:R_0402_1005Metric, F.Cu at (67.9, 138.7)
- added R429: 10k, Resistor_SMD:R_0402_1005Metric, F.Cu at (67.9, 140.7)
- added R430: 10k, Resistor_SMD:R_0402_1005Metric, F.Cu at (67.9, 142.6)
- added R431: 10k, Resistor_SMD:R_0402_1005Metric, F.Cu at (67.9, 144.6)
- added R432: 10k, Resistor_SMD:R_0402_1005Metric, F.Cu at (67.9, 146.6)
- added R433: 10k, Resistor_SMD:R_0402_1005Metric, F.Cu at (255.8, 141.6)
- added R434: 10k, Resistor_SMD:R_0402_1005Metric, F.Cu at (257.8, 141.6)
- added R435: 10k, Resistor_SMD:R_0402_1005Metric, F.Cu at (59.8, 55.7)
- added R436: 10k, Resistor_SMD:R_0402_1005Metric, F.Cu at (59.8, 57.7)
- added R437: 10k, Resistor_SMD:R_0402_1005Metric, F.Cu at (59.8, 59.7)
- added R438: 10k, Resistor_SMD:R_0402_1005Metric, F.Cu at (59.8, 61.7)
- added R439: 10k, Resistor_SMD:R_0402_1005Metric, F.Cu at (59.8, 63.7)
- added R440: 10k, Resistor_SMD:R_0402_1005Metric, F.Cu at (59.8, 65.7)
- added R441: 10k, Resistor_SMD:R_0402_1005Metric, F.Cu at (59.8, 67.7)
- added R442: 10k, Resistor_SMD:R_0402_1005Metric, F.Cu at (59.8, 69.7)
- added R443: 10k, Resistor_SMD:R_0402_1005Metric, F.Cu at (70.8, 136.7)
- added R444: 10k, Resistor_SMD:R_0402_1005Metric, F.Cu at (70.8, 138.7)
- added R445: 10k, Resistor_SMD:R_0402_1005Metric, F.Cu at (70.8, 140.7)
- added R446: 10k, Resistor_SMD:R_0402_1005Metric, F.Cu at (70.8, 142.6)
- added R447: 10k, Resistor_SMD:R_0402_1005Metric, F.Cu at (70.8, 144.6)
- added R448: 10k, Resistor_SMD:R_0402_1005Metric, F.Cu at (70.8, 146.6)
- added R449: 10k, Resistor_SMD:R_0402_1005Metric, F.Cu at (70.8, 148.6)
- added R450: 10k, Resistor_SMD:R_0402_1005Metric, F.Cu at (70.8, 150.6)
- added R451: 10k, Resistor_SMD:R_0402_1005Metric, F.Cu at (59.8, 71.7)
- added R452: 10k, Resistor_SMD:R_0402_1005Metric, F.Cu at (62.7, 55.7)
- added R453: 10k, Resistor_SMD:R_0402_1005Metric, F.Cu at (62.7, 57.7)
- added R454: 10k, Resistor_SMD:R_0402_1005Metric, F.Cu at (62.7, 59.7)
- added R455: 10k, Resistor_SMD:R_0402_1005Metric, F.Cu at (62.7, 61.7)
- added R456: 10k, Resistor_SMD:R_0402_1005Metric, F.Cu at (62.7, 63.7)
- added R457: 10k, Resistor_SMD:R_0402_1005Metric, F.Cu at (62.7, 65.7)
- added R458: 10k, Resistor_SMD:R_0402_1005Metric, F.Cu at (62.7, 67.7)
- added R459: 10k, Resistor_SMD:R_0402_1005Metric, F.Cu at (73.7, 136.7)
- added R460: 10k, Resistor_SMD:R_0402_1005Metric, F.Cu at (73.7, 138.7)
- added R461: 10k, Resistor_SMD:R_0402_1005Metric, F.Cu at (73.7, 140.7)
- added R462: 10k, Resistor_SMD:R_0402_1005Metric, F.Cu at (73.7, 142.6)
- added R463: 10k, Resistor_SMD:R_0402_1005Metric, F.Cu at (73.7, 144.6)
- added R464: 10k, Resistor_SMD:R_0402_1005Metric, F.Cu at (73.7, 146.6)
- added R465: 10k, Resistor_SMD:R_0402_1005Metric, F.Cu at (73.7, 148.6)
- added R466: 10k, Resistor_SMD:R_0402_1005Metric, F.Cu at (73.7, 150.6)
- added SW101: SW_Push, Library:SMT Push Button 12x12, F.Cu at (74.7, 61.4)
- added SW301: SW_Push, Button_Switch_SMD:SW_Push_1P1T_NO_6x6mm_H9.5mm, F.Cu at (71.7, 84.8)
- added SW302: SW_Push, Button_Switch_SMD:SW_Push_1P1T_NO_6x6mm_H9.5mm, F.Cu at (71.7, 92.4)
- added SW601: SW_SPDT, Library:472121010111, F.Cu at (165.4, 7.90)
- added U201: MOS6581/6582/8580SID, Package_DIP:DIP-28_W15.24mm_LongPads, F.Cu at (233.2, 65.2)
- RV514: footprint libs:Potentiometer_Alps_RK09K_Horizontal_CORRECTED -> libs:PTB6044-2010BPA103_BRN
- SW401, SW402, SW403: footprint Button_Switch_THT:SW_NKK_NR01 -> Library:S-2050
- U401: renamed from U402; moved to F.Cu
- moved C401 197.0 mm to (54.0, 73.6)
- moved C402 197.0 mm to (54.0, 75.6)
- moved C403 197.0 mm to (54.0, 77.6)
- moved S408 141.8 mm to (255.0, 150.0), turned to 0 degrees
- moved S401 140.4 mm to (115.0, 150.0), turned to 0 degrees
- moved SW402 135.8 mm to (45.5, 61.7)
- moved SW403 129.7 mm to (45.5, 75.7)
- moved U402 126.3 mm to (246.3, 129.1), turned to 0 degrees
- moved RV514 105.1 mm to (275.0, 185.0), turned to 90 degrees
- moved U404 104.2 mm to (151.4, 130.7), turned to 0 degrees
- moved S407 102.2 mm to (235.0, 150.0), turned to 0 degrees
- moved S402 100.8 mm to (135.0, 150.0), turned to 0 degrees
- moved U403 77.0 mm to (137.2, 129.9), turned to 0 degrees
- moved S406 63.2 mm to (215.0, 150.0), turned to 0 degrees
- moved S403 61.8 mm to (155.0, 150.0), turned to 0 degrees
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- renumbered C303 to C304, C304 to C305, C305 to C306, C306 to C307, C307 to C309, C308 to C310, H108 to H105, H107 to H106, H106 to H107, H105 to H108, S1 to S402, S2 to S403, S3 to S404, S4 to S405, S5 to S406, S6 to S407, S7 to S408, S8 to S409, S9 to S410, S10 to S411, S11 to S412, S12 to S413, S13 to S414, S14 to S415, S15 to S416, SW301 to SW303, U1 to U402, U401 to U403, U2 to U404, U602 to U601, U601 to U602
Connections:
- C401 pad 1: Net-(SW401-Common) -> /GPIO_Expandeur/B0
- C401 pad 2: +3.3V -> GND
- C402 pad 1: Net-(SW402-Common) -> /GPIO_Expandeur/B1
- C402 pad 2: +3.3V -> GND
- C403 pad 1: Net-(SW403-Common) -> /GPIO_Expandeur/B2
- C403 pad 2: +3.3V -> GND
- J301 pad 12: unconnected-(J301-~{RST}-Pad12) -> /STM32-G474RE/NRST
- J301 pad 13: unconnected-(J301-VCP_RX-Pad13) -> /STM32-G474RE/VCP_RX
- J301 pad 14: unconnected-(J301-VCP_TX-Pad14) -> /STM32-G474RE/VCP_TX
- J301 pad 4: unconnected-(J301-JTMS/SWDIO-Pad4) -> /STM32-G474RE/SWDIO
- J301 pad 6: unconnected-(J301-JCLK/SWCLK-Pad6) -> /STM32-G474RE/SWCLK
- J601 pad A4: +5V -> VBUS
- J601 pad A9: +5V -> VBUS
- J601 pad B4: +5V -> VBUS
- J601 pad B9: +5V -> VBUS
- S401 pad 1: /GPIO_Expandeur/B0 -> Net-(R403-Pad2)
- S401 pad 2: +3.3V -> GND
- S401 pad L2: Net-(R2-Pad2) -> unconnected-(S401-PadL2)
- S402 pad 1: /GPIO_Expandeur/B1 -> Net-(R404-Pad2)
- S402 pad 2: +3.3V -> GND
- S402 pad L2: Net-(R5-Pad2) -> unconnected-(S402-PadL2)
- S403 pad 1: /GPIO_Expandeur/B2 -> Net-(R405-Pad2)
- S403 pad 2: +3.3V -> GND
- S403 pad L2: Net-(R8-Pad2) -> unconnected-(S403-PadL2)
- S404 pad 1: /GPIO_Expandeur/B3 -> Net-(R406-Pad2)
- S404 pad 2: +3.3V -> GND
- S404 pad L2: Net-(R11-Pad2) -> unconnected-(S404-PadL2)
- S405 pad 1: /GPIO_Expandeur/B4 -> Net-(R419-Pad2)
- S405 pad 2: +3.3V -> GND
- S405 pad L2: Net-(R14-Pad2) -> unconnected-(S405-PadL2)
- S406 pad 1: /GPIO_Expandeur/B5 -> Net-(R420-Pad2)
- S406 pad 2: +3.3V -> GND
- S406 pad L2: Net-(R17-Pad2) -> unconnected-(S406-PadL2)
- S407 pad 1: /GPIO_Expandeur/B6 -> Net-(R421-Pad2)
- S407 pad 2: +3.3V -> GND
- S407 pad L2: Net-(R20-Pad2) -> unconnected-(S407-PadL2)
- S408 pad 1: /GPIO_Expandeur/B7 -> Net-(R422-Pad2)
- S408 pad 2: +3.3V -> GND
- S408 pad L2: Net-(R23-Pad2) -> unconnected-(S408-PadL2)
- S409 pad 1: /GPIO_Expandeur/B8 -> Net-(R435-Pad2)
- S409 pad 2: +3.3V -> GND
- S409 pad L2: Net-(R26-Pad2) -> unconnected-(S409-PadL2)
- S410 pad 1: /GPIO_Expandeur/B9 -> Net-(R436-Pad2)
- S410 pad 2: +3.3V -> GND
- S410 pad L2: Net-(R29-Pad2) -> unconnected-(S410-PadL2)
- S411 pad 1: /GPIO_Expandeur/B10 -> Net-(R437-Pad2)
- S411 pad 2: +3.3V -> GND
- S411 pad L2: Net-(R32-Pad2) -> unconnected-(S411-PadL2)
- S412 pad 1: /GPIO_Expandeur/B11 -> Net-(R438-Pad2)
- S412 pad 2: +3.3V -> GND
- S412 pad L2: Net-(R35-Pad2) -> unconnected-(S412-PadL2)
- S413 pad 1: /GPIO_Expandeur/B12 -> Net-(R451-Pad2)
- S413 pad 2: +3.3V -> GND
- S413 pad L2: Net-(R38-Pad2) -> unconnected-(S413-PadL2)
- S414 pad 1: /GPIO_Expandeur/B13 -> Net-(R452-Pad2)
- S414 pad 2: +3.3V -> GND
- S414 pad L2: Net-(R41-Pad2) -> unconnected-(S414-PadL2)
- S415 pad 1: /GPIO_Expandeur/B14 -> Net-(R453-Pad2)
- S415 pad 2: +3.3V -> GND
- S415 pad L2: Net-(R44-Pad2) -> unconnected-(S415-PadL2)
- S416 pad 1: /GPIO_Expandeur/B15 -> Net-(R454-Pad2)
- S416 pad 2: +3.3V -> GND
- S416 pad L2: Net-(R47-Pad2) -> unconnected-(S416-PadL2)
- SW401 pad C: Net-(SW401-Common) -> GND
- SW402 pad C: Net-(SW402-Common) -> GND
- SW403 pad C: Net-(SW403-Common) -> GND
- U301 pad 18: unconnected-(U301-PA4-Pad18) -> /STM32-G474RE/BTN_1
- U301 pad 19: unconnected-(U301-PA5-Pad19) -> /STM32-G474RE/BTN_2
- U301 pad 2: /MOS6581/A2 -> /STM32-G474RE/LED1
- U301 pad 22: /STM32-G474RE/I2C_2_SCL -> /STM32-G474RE/VCP_TX
- U301 pad 23: unconnected-(U301-PC5-Pad23) -> /STM32-G474RE/VCP_RX
- U301 pad 26: /MOS6581/D0 -> /STM32-G474RE/Tap_Tempo
- U301 pad 28: unconnected-(U301-VREF+-Pad28) -> +3.3V
- U301 pad 3: /MOS6581/A3 -> /STM32-G474RE/LED2
- U301 pad 35: unconnected-(U301-PB13-Pad35) -> /GPIO_Expandeur/INTA_2
- U301 pad 37: unconnected-(U301-PB15-Pad37) -> /GPIO_Expandeur/INTB_2
- U301 pad 38: unconnected-(U301-PC6-Pad38) -> /GPIO_Expandeur/INTB_1
- U301 pad 39: unconnected-(U301-PC7-Pad39) -> /GPIO_Expandeur/INTA_1
- U301 pad 4: /MOS6581/A4 -> /STM32-G474RE/LED3
- U301 pad 40: /GPIO_Expandeur/SDA Expandeur_Boutons -> /GPIO_Expandeur/I2C_SCL
- U301 pad 41: /GPIO_Expandeur/SCK Expandeur_Boutons -> /GPIO_Expandeur/I2C_SDA
- U301 pad 42: unconnected-(U301-PA8-Pad42) -> /MOS6581/MOS6581_Read/Write
- U301 pad 43: unconnected-(U301-PA9-Pad43) -> /MOS6581//Reset
- U301 pad 44: unconnected-(U301-PA10-Pad44) -> /MOS6581/A0
- U301 pad 49: /GPIO_Expandeur/SCK LED_Driver -> /STM32-G474RE/SWDIO
- U301 pad 5: /STM32-G474RE/I2C_2_SDA -> unconnected-(U301-PF0-Pad5)
- U301 pad 50: /GPIO_Expandeur/SDA LED_Driver -> /STM32-G474RE/SWCLK
- U301 pad 51: unconnected-(U301-PA15-Pad51) -> /MOS6581/A1
- U301 pad 52: unconnected-(U301-PC10-Pad52) -> /MOS6581/A2
- U301 pad 53: /MOS6581/A0 -> /MOS6581/A3
- U301 pad 54: /MOS6581/A1 -> /MOS6581/A4
- U301 pad 55: unconnected-(U301-PD2-Pad55) -> /MOS6581/D0
- U301 pad 7: unconnected-(U301-PG10-Pad7) -> Net-(U301-PG10)
- U401 pad 12: Net-(U401-GPA5) -> /GPIO_Expandeur/I2C_SCL
- U401 pad 13: Net-(U401-GPA4) -> /GPIO_Expandeur/I2C_SDA
- U401 pad 18: /GPIO_Expandeur/Reset -> +3.3V
- U401 pad 19: Net-(U401-GPA6) -> /GPIO_Expandeur/INTB_2
- U401 pad 20: Net-(U401-GPA7) -> /GPIO_Expandeur/INTA_2
- U402 pad 1: +3.3V -> GND
- U402 pad 10: /GPIO_Expandeur/B4_B -> /GPIO_Expandeur/B6_R
- U402 pad 11: /GPIO_Expandeur/B5_B -> /GPIO_Expandeur/B6_B
- U402 pad 12: /GPIO_Expandeur/B6_B -> /GPIO_Expandeur/B7_R
- U402 pad 16: /GPIO_Expandeur/B14_B -> /GPIO_Expandeur/B15_R
- U402 pad 17: /GPIO_Expandeur/B13_B -> /GPIO_Expandeur/B14_B
- U402 pad 18: /GPIO_Expandeur/B12_B -> /GPIO_Expandeur/B14_R
- U402 pad 19: /GPIO_Expandeur/B11_B -> /GPIO_Expandeur/B13_B
- U402 pad 2: +3.3V -> GND
- U402 pad 20: /GPIO_Expandeur/B10_B -> /GPIO_Expandeur/B13_R
- U402 pad 21: /GPIO_Expandeur/B9_B -> /GPIO_Expandeur/B12_B
- U402 pad 22: /GPIO_Expandeur/B8_B -> /GPIO_Expandeur/B12_R
- U402 pad 23: unconnected-(U1-~{OE}-Pad23) -> Net-(U402-~{OE})
- U402 pad 26: Net-(U1-SCL) -> /GPIO_Expandeur/I2C_SDA
- U402 pad 27: Net-(U1-SDA) -> /GPIO_Expandeur/I2C_SCL
- U402 pad 3: +3.3V -> GND
- U402 pad 4: +3.3V -> GND
- U402 pad 6: /GPIO_Expandeur/B0_B -> /GPIO_Expandeur/B4_R
- U402 pad 7: /GPIO_Expandeur/B1_B -> /GPIO_Expandeur/B4_B
- U402 pad 8: /GPIO_Expandeur/B2_B -> /GPIO_Expandeur/B5_R
- U402 pad 9: /GPIO_Expandeur/B3_B -> /GPIO_Expandeur/B5_B
- U403 pad 12: /GPIO_Expandeur/SCK Expandeur_Boutons -> /GPIO_Expandeur/I2C_SCL
- U403 pad 13: /GPIO_Expandeur/SDA Expandeur_Boutons -> /GPIO_Expandeur/I2C_SDA
- U403 pad 18: /GPIO_Expandeur/Reset -> +3.3V
- U403 pad 19: /GPIO_Expandeur/INTA_Boutons -> /GPIO_Expandeur/INTB_1
- U403 pad 20: /GPIO_Expandeur/INTB_Boutons -> /GPIO_Expandeur/INTA_1
- U403 pad 25: Net-(U401-GPA4) -> unconnected-(U403-GPA4-Pad25)
- U403 pad 26: Net-(U401-GPA5) -> unconnected-(U403-GPA5-Pad26)
- U403 pad 27: Net-(U401-GPA6) -> unconnected-(U403-GPA6-Pad27)
- U403 pad 28: Net-(U401-GPA7) -> unconnected-(U403-GPA7-Pad28)
- U404 pad 10: /GPIO_Expandeur/B4_R -> /GPIO_Expandeur/B2_R
- U404 pad 11: /GPIO_Expandeur/B5_R -> /GPIO_Expandeur/B2_B
- U404 pad 12: /GPIO_Expandeur/B6_R -> /GPIO_Expandeur/B3_R
- U404 pad 13: /GPIO_Expandeur/B7_R -> /GPIO_Expandeur/B3_B
- U404 pad 15: /GPIO_Expandeur/B8_R -> /GPIO_Expandeur/B11_B
- U404 pad 16: /GPIO_Expandeur/B9_R -> /GPIO_Expandeur/B11_R
- U404 pad 17: /GPIO_Expandeur/B10_R -> /GPIO_Expandeur/B10_B
- U404 pad 18: /GPIO_Expandeur/B11_R -> /GPIO_Expandeur/B10_R
- U404 pad 19: /GPIO_Expandeur/B12_R -> /GPIO_Expandeur/B9_B
- U404 pad 2: +3.3V -> GND
- U404 pad 20: /GPIO_Expandeur/B13_R -> /GPIO_Expandeur/B9_R
- U404 pad 21: /GPIO_Expandeur/B14_R -> /GPIO_Expandeur/B8_B
- U404 pad 22: /GPIO_Expandeur/B15_R -> /GPIO_Expandeur/B8_R
- U404 pad 23: unconnected-(U2-~{OE}-Pad23) -> Net-(U404-~{OE})
- U404 pad 26: Net-(U2-SCL) -> /GPIO_Expandeur/I2C_SDA
- U404 pad 27: Net-(U2-SDA) -> /GPIO_Expandeur/I2C_SCL
- U404 pad 3: +3.3V -> GND
- U404 pad 7: /GPIO_Expandeur/B1_R -> /GPIO_Expandeur/B0_B
- U404 pad 8: /GPIO_Expandeur/B2_R -> /GPIO_Expandeur/B1_R
- U404 pad 9: /GPIO_Expandeur/B3_R -> /GPIO_Expandeur/B1_B
- U602 pad 5: +5V -> VBUS
Routing:
- net /Potar/Voice2_PW_pot: track 73.3 -> 0.00 mm
- net /Potar/Voice1_PW_pot: track 72.6 -> 0.00 mm, vias 1 -> 0
- net /Potar/Voice1_Attack_pot: track 56.8 -> 0.00 mm
- net /Potar/Voice2_Attack_pot: track 56.1 -> 0.00 mm, vias 1 -> 0
- net +3.3V: track 64.8 -> 9.60 mm, vias 0 -> 16
- net /GPIO_Expandeur/B4_R: track 54.3 -> 0.00 mm
- net /Potar/Voice2_Decay_pot: track 40.5 -> 0.00 mm
- net /Potar/Voice1_Decay_pot: track 38.8 -> 0.00 mm, vias 1 -> 0
- net /Potar/Voice2_Release_pot: track 22.9 -> 0.00 mm, vias 1 -> 0
- net /Potar/Voice1_Release_pot: track 21.8 -> 0.00 mm
- net /GPIO_Expandeur/B6_B: track 18.8 -> 0.00 mm
- net /GPIO_Expandeur/B8_R: track 18.7 -> 0.00 mm
- net /GPIO_Expandeur/B8: track 18.4 -> 0.00 mm
- net Net-(R466-Pad2): track 23.4 -> 6.40 mm
- net VBUS: track 0.00 -> 15.8 mm
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
Commit message: PCB PCB PCB
Parts:
- moved J101 218.3 mm to (293.5, 64.2), turned to 180 degrees
- moved R454 216.1 mm to (250.6, 166.5)
- moved R458 214.0 mm to (252.5, 166.5), turned to 180 degrees
- moved C416 205.4 mm to (248.7, 166.5), turned to 180 degrees
- moved R453 200.1 mm to (230.7, 166.5)
- moved R457 197.6 mm to (232.6, 166.5), turned to 180 degrees
- moved SW101 196.7 mm to (271.3, 59.0)
- moved C308 191.4 mm to (256.5, 68.4), turned to 180 degrees
- moved R421 191.2 mm to (230.6, 141.5)
- moved C303 189.9 mm to (256.5, 77.6), turned to 180 degrees
- moved R425 189.8 mm to (232.5, 141.5), turned to 180 degrees
- moved C415 188.4 mm to (228.7, 166.5)
- moved C516 185.3 mm to (273.0, 88.6), turned to -90 degrees
- moved R466 184.8 mm to (257.8, 166.6), turned to 180 degrees
- moved R452 184.8 mm to (210.6, 166.5)
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Connections:
- C207 pad 2: GND -> /MOS6581/Audio_out
- J101 pad R1: GND -> /MOS6581/Audio_out
- J101 pad T: GND -> /MOS6581/Audio_out
Routing:
- net GND: track 14.6 -> 153.0 mm, vias 21 -> 68
- net /Potar/Filter_Res_pot: track 0.00 -> 112.3 mm, vias 0 -> 4
- net /Potar/Filter_Freq_pot: track 0.00 -> 75.8 mm, vias 0 -> 2
- net +3.3V: track 9.60 -> 85.3 mm, vias 16 -> 42
- net /MOS6581/D6: track 0.00 -> 62.6 mm, vias 0 -> 2
- net /Potar/Voice1_PW_pot: track 0.00 -> 62.4 mm
- net /MOS6581/D7: track 0.00 -> 62.1 mm, vias 0 -> 2
- net /MOS6581/D0: track 0.00 -> 61.9 mm, vias 0 -> 2
- net /MOS6581/D1: track 0.00 -> 61.8 mm, vias 0 -> 2
- net /Potar/Voice3_PW_pot: track 0.00 -> 60.8 mm
- net /MOS6581//Reset: track 0.00 -> 60.7 mm, vias 0 -> 2
- net /MOS6581/D4: track 0.00 -> 59.5 mm, vias 0 -> 2
- net /MOS6581/D3: track 0.00 -> 59.5 mm, vias 0 -> 2
- net /Potar/Voice2_PW_pot: track 0.00 -> 59.3 mm
- net /MOS6581/D2: track 0.00 -> 58.8 mm, vias 0 -> 2
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