File: Hardware/Sequencer/Sequencer.kicad_pcb (KiCad board)
At the start: 4 copper layers, 200 x 150 mm, 196 parts, among them J101 LINEOUT, J301 Conn_ST_STDC14, J601 USB_C_Receptacle_USB2.0_16P, SW101 SW_Push, SW301 SW_Push, SW302 SW_Push, SW303 SW_Push, SW401 SW_SP4T_NR01104, SW402 SW_SP4T_NR01104, SW403 SW_SP4T_NR01104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

Commit message: PCB uP bientot fini
Parts:
- added R1: 0, Resistor_SMD:R_0402_1005Metric, F.Cu at (246.4, 108.3)
- added R2: 0, Resistor_SMD:R_0402_1005Metric, F.Cu at (245.3, 108.3)
- added R3: 0, Resistor_SMD:R_0402_1005Metric, F.Cu at (253.4, 108.2)
- added R4: 0, Resistor_SMD:R_0402_1005Metric, F.Cu at (252.3, 108.2)
- moved RV514 85.6 mm to (285.0, 100.0), turned to -90 degrees
- moved SW303 44.2 mm to (240.2, 59.7)
- moved C514 27.9 mm to (288.0, 119.2), turned to -90 degrees
- moved C202 19.3 mm to (253.9, 109.9)
- moved C205 15.2 mm to (248.2, 111.3)
- moved C201 8.09 mm to (253.9, 111.2)
- moved C206 7.96 mm to (248.2, 110.2)
- moved C310 7.47 mm to (245.8, 59.8), turned to 90 degrees
- moved R303 4.01 mm to (217.5, 65.9), turned to 180 degrees
- moved RV516 3.00 mm to (271.6, 89.7)
- moved C302 0.92 mm to (204.2, 66.7)
Connections:
- C205 pad 1: +12V -> +5V
- C206 pad 1: +12V -> +5V
- U201 pad 25: +5V -> Net-(U201-VCC)
- U201 pad 28: +12V -> Net-(U201-VDD)
Routing:
- net +5V: track 9.72 -> 152.8 mm, vias 0 -> 2
- net /Potar/Voice1_Decay_pot: track 29.5 -> 130.2 mm, vias 0 -> 6
- net /Potar/Pitch_Main_pot: track 0.00 -> 96.0 mm, vias 0 -> 3
- net GND: track 153.0 -> 237.8 mm, vias 68 -> 71
- net /Potar/Voice3_PW_pot: track 60.8 -> 141.1 mm, vias 0 -> 2
- net /Potar/Voice3_Attack_pot: track 43.5 -> 122.9 mm, vias 0 -> 2
- net /Potar/Voice3_Decay_pot: track 25.7 -> 102.7 mm, vias 0 -> 2
- net /STM32-G474RE/SWCLK: track 0.00 -> 71.7 mm, vias 0 -> 4
- net /STM32-G474RE/SWDIO: track 0.00 -> 60.4 mm, vias 0 -> 4
- net /STM32-G474RE/BTN_2: track 2.41 -> 61.9 mm, vias 0 -> 2
- net Net-(U201-AUDIO_OUT): track 2.61 -> 59.0 mm
- net /STM32-G474RE/Tap_Tempo: track 2.53 -> 58.3 mm, vias 0 -> 2
- net /Potar/Voice2_Release_pot: track 6.98 -> 60.2 mm, vias 0 -> 2
- net /Potar/Voice1_Release_pot: track 8.13 -> 51.8 mm, vias 0 -> 4
- net /STM32-G474RE/VCP_RX: track 0.00 -> 43.5 mm, vias 0 -> 2
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