File: Hardware/Sequencer/MOS6581.kicad_sch (KiCad schematic)
At the start: 7 parts, among them U201 MOS6581/6582/8580SID

Commit message: Beaucoup de changements sur le pcb
Alim corrigée, ajout de l'USB C

Sonde sur le processeur + linkage USB

Rajout des boutons (465M111...)
Parts:
- added C207: 1u, symbol Device:C_Small
- added R201: 1k, symbol Device:R_Small
- renumbered C203 to C201, C204 to C202, C201 to C203, C202 to C204
Connections:
- net GND: now also U201.8 (/CS), C207.2, R201.2
- net Reset: now reaches U201.5 (/RES)
- net CLK_1MHZ: now reaches U201.6 (PHI2)
- net MOS6581_Read/Write: now reaches U201.7 (R/W)
- net AUDIO_OUT: no longer names the net of U201.27 (AUDIO_OUT)
- net AUDIO_OUT: now also C207.1, R201.1
- no-connect marks 0 -> 3

Commit message: update dimension pcb, footprint
Parts:
- C202, C203, C204, C205, C206, C207: footprint (none) -> Capacitor_SMD:C_0402_1005Metric
- R201: footprint (none) -> Resistor_SMD:R_0402_1005Metric
Changed lines of the file:
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@@
 			)
 		)
-		(property "Footprint" ""
+		(property "Footprint" "Capacitor_SMD:C_0402_1005Metric"
 			(at 207.01 78.74 0)
 			(effects
@@
 			)
 		)
-		(property "Footprint" ""
+		(property "Footprint" "Capacitor_SMD:C_0402_1005Metric"
 			(at 124.46 100.33 0)
 			(effects
@@
 			)
 		)
-		(property "Footprint" ""
+		(property "Footprint" "Resistor_SMD:R_0402_1005Metric"
 			(at 196.85 81.28 0)
 			(effects
@@
 			)
 		)
-		(property "Footprint" ""
+		(property "Footprint" "Capacitor_SMD:C_0402_1005Metric"
 			(at 115.57 41.91 0)
 			(effects
@@
 			)
 		)
-		(property "Footprint" ""
+		(property "Footprint" "Capacitor_SMD:C_0402_1005Metric"
 			(at 124.46 90.17 0)
 			(effects
@@
 			)
 		)
-		(property "Footprint" ""
+		(property "Footprint" "Capacitor_SMD:C_0402_1005Metric"
 			(at 143.51 41.91 0)
 			(effects
@@
 			)
 		)
-		(property "Footprint" ""
+		(property "Footprint" "Capacitor_SMD:C_0402_1005Metric"
 			(at 133.35 41.91 0)
 			(effects

Commit message: much changes everywhere
Changed lines of the file:
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@@
 		(at 176.53 87.63)
+	)
+	(bus_entry
+		(at 143.51 43.18)
+		(size 2.54 2.54)
+		(stroke
+			(width 0)
+			(type default)
+		)
 	)
 	(wire

Commit message: pcb
Changed lines of the file:
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@@
+		)
+	)
+	(hierarchical_label "Audio_out"
+		(shape input)
+		(at 209.55 78.74 0)
+		(fields_autoplaced yes)
+		(effects
+			(font
+				(size 1.27 1.27)
+			)
+			(justify left)
 		)
 	)

Commit message: update pcb
Parts:
- U201: footprint Housings_DIP:DIP-28_W15.24mm_Socket -> Package_DIP:DIP-28_W15.24mm_LongPads
Connections:
- net Reset renamed /Reset
Changed lines of the file:
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@@
 		(at 176.53 87.63)
-	)
-	(bus_entry
-		(at 143.51 43.18)
-		(size 2.54 2.54)
-		(stroke
-			(width 0)
-			(type default)
-		)
 	)
 	(wire
@@
 		)
 	)
-	(hierarchical_label "Reset"
+	(hierarchical_label "{slash}Reset"
 		(shape input)
 		(at 133.35 109.22 180)
@@
 			)
 		)
-		(property "Footprint" "Housings_DIP:DIP-28_W15.24mm_Socket"
+		(property "Footprint" "Package_DIP:DIP-28_W15.24mm_LongPads"
 			(at 154.94 128.27 0)
 			(effects

Commit message: PCB PCB PCB
Connections:
- net GND: no longer C207.2
- new net Audio_out: C207.2
Changed lines of the file:
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@@
-	)
-	(junction
-		(at 209.55 83.82)
-		(diameter 0)
-		(color 0 0 0 0)
 	)
 	(junction
@@
 		)
 		(stroke
-			(width 0)
-			(type default)
-		)
-	)
-	(wire
-		(pts
-			(xy 209.55 78.74) (xy 209.55 83.82)
-		)
-		(stroke

Commit message: PCB uP bientot fini
Parts:
- added R1, R2, R3, R4: 0, Resistor_SMD:R_0402_1005Metric, symbol Device:R_Small
Connections:
- net +5V: now also C205.1, C206.1, R1.1, R3.1; no longer U201.25 (VCC)
- removed net +12V: C205.1, C206.1, U201.28 (VDD)
- new net: R1.2, R2.2, U201.25 (VCC)
- new net: R3.2, R4.2, U201.28 (VDD)
- new net +3.3V: R2.1, R4.1
