File: Hardware/Sequencer/GPIO_Expandeur.kicad_sch (KiCad schematic)
At the start: 9 parts, among them SW401 SW_SP4T_NR01104, SW402 SW_SP4T_NR01104, SW403 SW_SP4T_NR01104, U401 MCP23017_SP, U402 MCP23017_SP

Commit message: GPIO
Parts:
- removed RV401, RV402, RV403, RV404: 10k, symbol Device:R_Potentiometer
- added C1, C2, C3: 10n, symbol Device:C_Small
Connections:
- net +3.3V: now also C1.2, C2.2, C3.2; no longer SW401.C (Common), SW402.C (Common), SW403.C (Common)
- net BUTTON1 renamed B0
- net BUTTON10 renamed A1
- net BUTTON11 renamed A2
- net BUTTON12 renamed A3
- net BUTTON13 renamed A4
- net BUTTON14 renamed A5
- net BUTTON15 renamed A6
- net BUTTON16 renamed A7
- net BUTTON2 renamed B1
- net BUTTON3 renamed B2
- net BUTTON4 renamed B3
- net BUTTON5 renamed B4
- net BUTTON6 renamed B5
- net BUTTON7 renamed B6
- net BUTTON8 renamed B7
- net BUTTON9 renamed A0
- new net: C2.1, SW402.C (Common)
- new net: C3.1, SW403.C (Common)
- new net: SW401.4, U401.1 (GPB0)
- new net: SW401.3, U401.2 (GPB1)
- new net: SW401.2, U401.3 (GPB2)
- new net: SW401.1, U401.4 (GPB3)
- new net: C1.1, SW401.C (Common)
Other:
- moved on the sheet: SW401

Commit message: Beaucoup de changements sur le pcb
Alim corrigée, ajout de l'USB C

Sonde sur le processeur + linkage USB

Rajout des boutons (465M111...)
Parts:
- added S401, S402, S403, S404, S405, S406, S407, S408, S409, S410, S411, S412, S413, S414, S415, S416: 465M111172501, 465M111172501:465M111172501, symbol 465M111172501:465M111172501
- renumbered C2 to C401, C3 to C402, C1 to C403, SW402 to SW401, SW403 to SW402, SW401 to SW403
Connections:
- net +3.3V: now also U401.15 (A0), U401.9 (VDD), U402.9 (VDD)
- net GND: now also U401.10 (VSS), U401.16 (A1), U401.17 (A2), U402.10 (VSS), U402.15 (A0), U402.16 (A1), U402.17 (A2)

Commit message: update dimension pcb, footprint
Parts:
- C401, C402, C403: footprint (none) -> Capacitor_SMD:C_0402_1005Metric
- U401, U402: footprint Package_DIP:DIP-28_W7.62mm -> Package_SO:SOIC-28W_7.5x17.9mm_P1.27mm; MPN (none) -> MCP23017-E/SO
Changed lines of the file:
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@@
 	)
 	(symbol
+		(lib_id "Interface_Expansion:MCP23017_SP")
+		(at 77.47 138.43 0)
+		(unit 1)
+		(exclude_from_sim no)
+		(in_bom yes)
+		(on_board yes)
+		(dnp no)
+		(fields_autoplaced yes)
+		(property "Reference" "U401"
+			(at 79.6641 110.49 0)
+			(effects
+				(font
+					(size 1.27 1.27)
+				)
+				(justify left)
+			)
+		)
+		(property "Value" "MCP23017_SP"
+			(at 79.6641 113.03 0)
+			(effects
+				(font
+					(size 1.27 1.27)
+				)
+				(justify left)
+			)
+		)
+		(property "Footprint" "Package_SO:SOIC-28W_7.5x17.9mm_P1.27mm"
+			(at 82.55 163.83 0)
+			(effects
+				(font
+					(size 1.27 1.27)
+				)
+				(justify left)
+				(hide yes)
+			)
+		)
+		(property "Datasheet" "https://ww1.microchip.com/downloads/en/devicedoc/20001952c.pdf"
+			(at 82.55 166.37 0)
+			(effects
+				(font
+					(size 1.27 1.27)
+				)
+				(justify left)
+				(hide yes)
+			)
+		)
+		(property "Description" "16-bit I/O expander, I2C, interrupts, w pull-ups, SPDIP-28"
+			(at 77.47 138.43 0)
+			(effects
+				(font
+					(size 1.27 1.27)
+				)
+				(hide yes)
+			)
+		)
+		(property "MPN" "MCP23017-E/SO"
+			(at 77.47 138.43 0)
+			(effects
+				(font
+					(size 1.27 1.27)
+				)
+				(hide yes)
+			)
+		)
+		(pin "28"
+		)
+		(pin "11"
+		)
+		(pin "3"
+		)
+		(pin "4"
+		)
+		(pin "12"
+		)
+		(pin "6"
+		)
+		(pin "19"
+		)
+		(pin "7"
+		)
+		(pin "9"
+		)
+		(pin "5"
+		)
+		(pin "10"
+		)
+		(pin "17"
+		)
+		(pin "15"
+		)
+		(pin "25"
+		)
+		(pin "20"
+		)
+		(pin "8"
+		)
+		(pin "1"
+		)
+		(pin "13"
+		)
+		(pin "14"
+		)
+		(pin "18"
+		)
+		(pin "2"
+		)
+		(pin "21"
+		)
+		(pin "22"
+		)
+		(pin "16"
+		)
+		(pin "23"
+		)
+		(pin "24"
+		)
+		(pin "26"
+		)
+		(pin "27"
+		)
+		(instances
+			(project "Sequencer"
+				(path "/bb3f736c-029c-4f1c-9c8c-1e3d4a336366/a53cf5d6-7d76-4909-bc26-231937405e3c"
+					(reference "U401")
+					(unit 1)
+				)
+			)
+		)
+	)
+	(symbol
 		(lib_id "Device:C_Small")
 		(at 115.57 130.81 90)
@@
 			)
 		)
-		(property "Footprint" ""
+		(property "Footprint" "Capacitor_SMD:C_0402_1005Metric"
 			(at 115.57 130.81 0)
 			(effects
@@
 			)
 		)
-		(property "Footprint" ""
+		(property "Footprint" "Capacitor_SMD:C_0402_1005Metric"
 			(at 115.57 143.51 0)
 			(effects
@@
 			)
 		)
-		(property "Footprint" "Package_DIP:DIP-28_W7.62mm"
+		(property "Footprint" "Package_SO:SOIC-28W_7.5x17.9mm_P1.27mm"
 			(at 104.14 78.74 0)
 			(effects
@@
 			)
 		)
-		(property "Datasheet" "http://ww1.microchip.com/downloads/en/DeviceDoc/20001952C.pdf"
+		(property "Datasheet" "https://ww1.microchip.com/downloads/en/devicedoc/20001952c.pdf"
 			(at 104.14 81.28 0)
 			(effects
@@
 			)
 		)
+		(property "MPN" "MCP23017-E/SO"
+			(at 99.06 53.34 0)
+			(effects
+				(font
+					(size 1.27 1.27)
+				)
+				(hide yes)
+			)
+		)
 		(pin "28"
 		)
@@
 	)
 	(symbol
-		(lib_id "Interface_Expansion:MCP23017_SP")
-		(at 77.47 138.43 0)
-		(unit 1)
-		(exclude_from_sim no)
-		(in_bom yes)
-		(on_board yes)
-		(dnp no)
-		(fields_autoplaced yes)
-		(property "Reference" "U401"
-			(at 79.6641 110.49 0)
-			(effects
-				(font
-					(size 1.27 1.27)
-				)
-				(justify left)
-			)
-		)
-		(property "Value" "MCP23017_SP"
-			(at 79.6641 113.03 0)
-			(effects
-				(font
-					(size 1.27 1.27)
-				)
-				(justify left)
-			)
-		)
-		(property "Footprint" "Package_DIP:DIP-28_W7.62mm"
-			(at 82.55 163.83 0)
-			(effects
-				(font
-					(size 1.27 1.27)
-				)
-				(justify left)
-				(hide yes)
-			)
-		)
-		(property "Datasheet" "http://ww1.microchip.com/downloads/en/DeviceDoc/20001952C.pdf"
-			(at 82.55 166.37 0)
-			(effects
-				(font
-					(size 1.27 1.27)
-				)
-				(justify left)
-				(hide yes)
-			)
-		)
-		(property "Description" "16-bit I/O expander, I2C, interrupts, w pull-ups, SPDIP-28"
-			(at 77.47 138.43 0)
-			(effects
-				(font
-					(size 1.27 1.27)
-				)
-				(hide yes)
-			)
-		)
-		(pin "28"
-		)
-		(pin "11"
-		)
-		(pin "3"
-		)
-		(pin "4"
-		)
-		(pin "12"
-		)
-		(pin "6"
-		)
-		(pin "19"
-		)
-		(pin "7"
-		)
-		(pin "9"
-		)
-		(pin "5"
-		)
-		(pin "10"
-		)
-		(pin "17"
-		)
-		(pin "15"
-		)
-		(pin "25"
-		)
-		(pin "20"
-		)
-		(pin "8"
-		)
-		(pin "1"
-		)
-		(pin "13"
-		)
-		(pin "14"
-		)
-		(pin "18"
-		)
-		(pin "2"
-		)
-		(pin "21"
-		)
-		(pin "22"
-		)
-		(pin "16"
-		)
-		(pin "23"
-		)
-		(pin "24"
-		)
-		(pin "26"
-		)
-		(pin "27"
-		)
-		(instances
-			(project "Sequencer"
-				(path "/bb3f736c-029c-4f1c-9c8c-1e3d4a336366/a53cf5d6-7d76-4909-bc26-231937405e3c"
-					(reference "U401")
-					(unit 1)
-				)
-			)
-		)
-	)
-	(symbol
 		(lib_id "power:+3.3V")
 		(at 121.92 130.81 270)
@@
 			)
 		)
-		(property "Footprint" ""
+		(property "Footprint" "Capacitor_SMD:C_0402_1005Metric"
 			(at 121.92 110.49 0)
 			(effects

Commit message: much changes everywhere
Parts:
- removed S402, S403, S404, S405, S406, S407, S408, S409, S410, S411, S412, S413, S414, S415, S416: 465M111172501, 465M111172501:465M111172501, symbol 465M111172501:465M111172501
- added C1, C10, C11, C12, C13, C14, C15, C16, C2, C3, C4, C5, C6, C7, C8, C9: 100n, symbol Device:C_Small
- added R1, R10, R11, R12, R13, R14, R15, R16, R17, R18, R19, R2, R20, R21, R22, R23, R24, R25, R26, R27, R28, R29, R3, R30, R31, R32, R33, R34, R35, R36, R37, R38, R39, R4, R40, R41, R42, R43, R44, R45, R46, R47, R48, R5, R6, R7, R8, R9: 10k, symbol Device:R_Small
- added S1, S10, S11, S12, S13, S14, S15, S2, S3, S4, S5, S6, S7, S8, S9: 465M111172501, libs:465M111172501, symbol 465M111172501:465M111172501
- added U1, U2: PCA9635, Package_SO:TSSOP-28_4.4x9.7mm_P0.65mm, symbol Driver_LED:PCA9635
- added U4: MCP23017_SP, Package_SO:SOIC-28W_7.5x17.9mm_P1.27mm, symbol Interface_Expansion:MCP23017_SP
- S401: footprint 465M111172501:465M111172501 -> libs:465M111172501
Connections:
- net +3.3V: now also S401.2, S401.LC, C1.1, C10.1, C11.1, C12.1, C13.1, C14.1, C15.1, C16.1, C2.1, C3.1, C4.1, C5.1, C6.1, C7.1, C8.1, C9.1, S1.2, S1.LC, S10.2, S10.LC, S11.2, S11.LC, S12.2, S12.LC, S13.2, S13.LC, S14.2, S14.LC, S15.2, S15.LC, S2.2, S2.LC, S3.2, S3.LC, S4.2, S4.LC, S5.2, S5.LC, S6.2, S6.LC, S7.2, S7.LC, S8.2, S8.LC, S9.2, S9.LC, U1.1 (A0), U1.2 (A1), U1.28 (VDD), U1.3 (A2), U1.4 (A3), U2.1 (A0), U2.2 (A1), U2.28 (VDD), U2.3 (A2), U4.16 (A1), U4.9 (VDD)
- net B0: now also S401.1, C1.2
- net B1: now also C2.2, S1.1
- net B2: now also C3.2, S2.1
- net B3: now also C4.2, S3.1
- net B4: now also C5.2, S4.1
- net B5: now also C6.2, S5.1
- net B6: now also C7.2, S6.1
- net B7: now also C8.2, S7.1
- net GND: now also U1.14 (VSS), U1.24 (A5), U1.25 (A6), U1.5 (A4), U2.14 (VSS), U2.24 (A5), U2.25 (A6), U2.4 (A3), U2.5 (A4), U4.10 (VSS), U4.15 (A0), U4.17 (A2)
- net SCK Expandeur_Boutons: now reaches U401.12 (SCK)
- net SDA Expandeur_Boutons: now reaches U401.13 (SDA)
- net Reset: now reaches U401.18 (~{RESET})
- net Reset: now also U402.18 (~{RESET}), U4.18 (~{RESET})
- net INTA_Boutons: now reaches U401.19 (INTB)
- net INTB_Boutons: now reaches U401.20 (INTA)
- net at U401.25 (GPA4): now also U402.13 (SDA)
- net at U401.26 (GPA5): now also U402.12 (SCK)
- net at U401.27 (GPA6): now also U402.19 (INTB)
- net at U401.28 (GPA7): now also U402.20 (INTA)
- net at S401.L1: now also R1.2
- net at S401.L2: now also R2.2
- net at S401.L3: now also R3.2
- new net: R28.2, S9.L1
- new net: R43.2, S14.L1
- new net: R47.2, S15.L2
- new net: R31.2, S10.L1
- new net: R32.2, S10.L2
- new net: R33.2, S10.L3
- new net: R38.2, S12.L2
- new net: R9.2, S2.L3
- new net: R29.2, S9.L2
- new net: R30.2, S9.L3
- new net: R15.2, S4.L3
- new net: R46.2, S15.L1
- new net: R19.2, S6.L1
- new net: R7.2, S2.L1
- new net: R8.2, S2.L2
- new net: R42.2, S13.L3
- new net: R25.2, S8.L1
- new net: R26.2, S8.L2
- new net: R27.2, S8.L3
- new net: R5.2, S1.L2
- new net: R37.2, S12.L1
- new net: R13.2, S4.L1
- new net: R22.2, S7.L1
- new net: U1.26 (SCL), U4.7 (GPB6)
- new net: U1.27 (SDA), U4.8 (GPB7)
- new net: U2.26 (SCL), U4.1 (GPB0)
- new net: U2.27 (SDA), U4.2 (GPB1)
- new net: R23.2, S7.L2
- new net: R41.2, S13.L2
- new net: R10.2, S3.L1
- new net: R11.2, S3.L2
- new net: R12.2, S3.L3
- new net: R39.2, S12.L3
- new net: R20.2, S6.L2
- new net: R40.2, S13.L1
- new net: R14.2, S4.L2
- new net: R48.2, S15.L3
- new net: R44.2, S14.L2
- new net: R45.2, S14.L3
- new net: R34.2, S11.L1
- new net: R16.2, S5.L1
- new net: R17.2, S5.L2
- new net: R18.2, S5.L3
- new net: R35.2, S11.L2
- new net: R36.2, S11.L3
- new net: R24.2, S7.L3
- new net: R6.2, S1.L3
- new net: R4.2, S1.L1
- new net: R21.2, S6.L3
- new net B0_B: R3.1, U1.6 (LED0)
- new net B0_G: R2.1
- new net B0_R: R1.1, U2.6 (LED0)
- new net B10: C11.2, S10.1
- new net B10_B: R33.1, U1.17 (LED10)
- new net B10_G: R32.1
- new net B10_R: R31.1, U2.17 (LED10)
- new net B11: C12.2, S11.1
- new net B11_B: R36.1, U1.18 (LED11)
- new net B11_G: R35.1
- new net B11_R: R34.1, U2.18 (LED11)
- new net B12: C13.2, S12.1
- new net B12_B: R39.1, U1.19 (LED12)
- new net B12_G: R38.1
- new net B12_R: R37.1, U2.19 (LED12)
- new net B13: C14.2, S13.1
- new net B13_B: R42.1, U1.20 (LED13)
- new net B13_G: R41.1
- new net B13_R: R40.1, U2.20 (LED13)
- new net B14: C15.2, S14.1
- new net B14_B: R45.1, U1.21 (LED14)
- new net B14_G: R44.1
- new net B14_R: R43.1, U2.21 (LED14)
- new net B15: C16.2, S15.1
- new net B15_B: R48.1, U1.22 (LED15)
- new net B15_G: R47.1
- new net B15_R: R46.1, U2.22 (LED15)
- new net B1_B: R6.1, U1.7 (LED1)
- new net B1_G: R5.1
- new net B1_R: R4.1, U2.7 (LED1)
- new net B2_B: R9.1, U1.8 (LED2)
- new net B2_G: R8.1
- new net B2_R: R7.1, U2.8 (LED2)
- new net B3_B: R12.1, U1.9 (LED3)
- new net B3_G: R11.1
- new net B3_R: R10.1, U2.9 (LED3)
- new net B4_B: R15.1, U1.10 (LED4)
- new net B4_G: R14.1
- new net B4_R: R13.1, U2.10 (LED4)
- new net B5_B: R18.1, U1.11 (LED5)
- new net B5_G: R17.1
- new net B5_R: R16.1, U2.11 (LED5)
- new net B6_B: R21.1, U1.12 (LED6)
- new net B6_G: R20.1
- new net B6_R: R19.1, U2.12 (LED6)
- new net B7_B: R24.1, U1.13 (LED7)
- new net B7_G: R23.1
- new net B7_R: R22.1, U2.13 (LED7)
- new net B8: C9.2, S8.1
- new net B8_B: R27.1, U1.15 (LED8)
- new net B8_G: R26.1
- new net B8_R: R25.1, U2.15 (LED8)
- new net B9: C10.2, S9.1
- new net B9_B: R30.1, U1.16 (LED9)
- new net B9_G: R29.1
- new net B9_R: R28.1, U2.16 (LED9)
- new net SCK LED_Driver: U4.12 (SCK)
- new net SDA LED_Driver: U4.13 (SDA)
- no-connect marks 0 -> 2
Other:
- note added: "GPIO EXPANDEUR SWITCH4 + BTNS"
- moved on the sheet: C401, C402, C403, S401, SW401, SW403, U401, U402

Commit message: pcb
Parts:
- C1, C10, C11, C12, C13, C14, C15, C16, C2, C3, C4, C5, C6, C7, C8, C9: footprint (none) -> Capacitor_SMD:C_0402_1005Metric
- R1, R10, R11, R12, R13, R14, R15, R16, R17, R18, R19, R2, R20, R21, R22, R23, R24, R25, R26, R27, R28, R29, R3, R30, R31, R32, R33, R34, R35, R36, R37, R38, R39, R4, R40, R41, R42, R43, R44, R45, R46, R47, R48, R5, R6, R7, R8, R9: footprint (none) -> Resistor_SMD:R_0402_1005Metric
Connections:
- net A0 is gone; now on net B8: U402.21 (GPA0)
- net A1 is gone; now on net B9: U402.22 (GPA1)
- net A2 is gone; now on net B10: U402.23 (GPA2)
- net A3 is gone; now on net B11: U402.24 (GPA3)
- net A4 is gone; now on net B12: U402.25 (GPA4)
- net A5 is gone; now on net B13: U402.26 (GPA5)
- net A6 is gone; now on net B14: U402.27 (GPA6)
- net A7 is gone; now on net B15: U402.28 (GPA7)
- net B10_B: now also U1.20 (LED13); no longer U1.17 (LED10)
- net B11_B: now also U1.19 (LED12); no longer U1.18 (LED11)
- net B12_B: now also U1.18 (LED11); no longer U1.19 (LED12)
- net B13_B: now also U1.17 (LED10); no longer U1.20 (LED13)
- net B14_B: now also U1.16 (LED9); no longer U1.21 (LED14)
- net B15_B: now also U1.15 (LED8); no longer U1.22 (LED15)
- net B8_B: now also U1.22 (LED15); no longer U1.15 (LED8)
- net B9_B: now also U1.21 (LED14); no longer U1.16 (LED9)
Other:
- note added: "Inverser 8-a-15"

Commit message: SCHEMA CORRECTION LED
Parts:
- removed R11, R14, R17, R2, R20, R23, R26, R29, R32, R35, R38, R41, R44, R47, R5, R8: 10k, Resistor_SMD:R_0402_1005Metric, symbol Device:R_Small
- removed U4: MCP23017_SP, Package_SO:SOIC-28W_7.5x17.9mm_P1.27mm, symbol Interface_Expansion:MCP23017_SP
Connections:
- net B0_B: now also U2.7 (LED1); no longer U1.6 (LED0)
- net B10_B: now also U2.17 (LED10); no longer U1.20 (LED13)
- net B10_R: now also U2.18 (LED11); no longer U2.17 (LED10)
- net B11_B: now also U2.15 (LED8); no longer U1.19 (LED12)
- net B11_R: now also U2.16 (LED9); no longer U2.18 (LED11)
- net B12_B: now also U1.21 (LED14); no longer U1.18 (LED11)
- net B12_R: now also U1.22 (LED15); no longer U2.19 (LED12)
- net B13_B: now also U1.19 (LED12); no longer U1.17 (LED10)
- net B13_R: now also U1.20 (LED13); no longer U2.20 (LED13)
- net B14_B: now also U1.17 (LED10); no longer U1.16 (LED9)
- net B14_R: now also U1.18 (LED11); no longer U2.21 (LED14)
- net B15_R: now also U1.16 (LED9); no longer U2.22 (LED15)
- net B1_B: now also U2.9 (LED3); no longer U1.7 (LED1)
- net B1_R: now also U2.8 (LED2); no longer U2.7 (LED1)
- net B2_B: now also U2.11 (LED5); no longer U1.8 (LED2)
- net B2_R: now also U2.10 (LED4); no longer U2.8 (LED2)
- net B3_B: now also U2.13 (LED7); no longer U1.9 (LED3)
- net B3_R: now also U2.12 (LED6); no longer U2.9 (LED3)
- net B4_B: now also U1.7 (LED1); no longer U1.10 (LED4)
- net B4_R: now also U1.6 (LED0); no longer U2.10 (LED4)
- net B5_B: now also U1.9 (LED3); no longer U1.11 (LED5)
- net B5_R: now also U1.8 (LED2); no longer U2.11 (LED5)
- net B6_B: now also U1.11 (LED5); no longer U1.12 (LED6)
- net B6_R: now also U1.10 (LED4); no longer U2.12 (LED6)
- net B7_R: now also U1.12 (LED6); no longer U2.13 (LED7)
- net B8_B: now also U2.21 (LED14); no longer U1.22 (LED15)
- net B8_R: now also U2.22 (LED15); no longer U2.15 (LED8)
- net B9_B: now also U2.19 (LED12); no longer U1.21 (LED14)
- net B9_R: now also U2.20 (LED13); no longer U2.16 (LED9)
- net SCL_4_7_15_12: now reaches U1.26 (SCL)
- net SDA_4_7_15_12: now reaches U1.27 (SDA)
- net SCL_0_3_11_8: now reaches U2.26 (SCL)
- net SDA_0_3_11_8: now reaches U2.27 (SDA)
- no-connect marks 2 -> 16

Commit message: update pcb
Parts:
- removed C1, C10, C11, C12, C13, C14, C15, C16, C2, C3, C4, C5, C6, C7, C8, C9: 100n, Capacitor_SMD:C_0402_1005Metric, symbol Device:C_Small
- added C404, C405, C406, C407, C408, C409, C410, C411, C412, C413, C414, C415, C416: 10n, Capacitor_SMD:C_0402_1005Metric, symbol Device:C_Small
- added R401, R402: 0, Resistor_SMD:R_0402_1005Metric, symbol Device:R_Small
- added R403, R404, R405, R406, R407, R408, R409, R410, R419, R420, R421, R422, R423, R424, R425, R426, R435, R436, R437, R438, R439, R440, R441, R442, R451, R452, R453, R454, R455, R456, R457, R458: 10k, Resistor_SMD:R_0402_1005Metric, symbol Device:R_Small
- SW401, SW402, SW403: footprint Button_Switch_THT:SW_NKK_NR01 -> Library:S-2050
- renumbered R1 to R411, R3 to R412, R4 to R413, R6 to R414, R7 to R415, R9 to R416, R10 to R417, R12 to R418, R13 to R427, R15 to R428, R16 to R429, R18 to R430, R19 to R431, R21 to R432, R22 to R433, R24 to R434, R25 to R443, R27 to R444, R28 to R445, R30 to R446, R31 to R447, R33 to R448, R34 to R449, R36 to R450, R37 to R459, R39 to R460, R40 to R461, R42 to R462, R43 to R463, R45 to R464, R46 to R465, R48 to R466, S1 to S402, S2 to S403, S3 to S404, S4 to S405, S5 to S406, S6 to S407, S7 to S408, S8 to S409, S9 to S410, S10 to S411, S11 to S412, S12 to S413, S13 to S414, S14 to S415, S15 to S416, U402 to U401, U1 to U402, U401 to U403, U2 to U404
Connections:
- net Reset is gone; now on net +3.3V: U401.18 (~{RESET}), U403.18 (~{RESET})
- net SCL_4_7_15_12 is gone; now on net I2C_SDA: U402.26 (SCL)
- net SDA Expandeur_Boutons is gone; now on net I2C_SDA: U403.13 (SDA)
- net SDA_0_3_11_8 is gone; now on net I2C_SCL: U404.27 (SDA)
- net SDA_4_7_15_12 is gone; now on net I2C_SCL: U402.27 (SDA)
- net +3.3V: now also R407.1, R408.1, R409.1, R410.1, R423.1, R424.1, R425.1, R426.1, R439.1, R440.1, R441.1, R442.1, R455.1, R456.1, R457.1, R458.1; no longer C401.2, C402.2, C403.2, S401.2, S402.2, S403.2, S404.2, S405.2, S406.2, S407.2, S408.2, S409.2, S410.2, S411.2, S412.2, S413.2, S414.2, S415.2, S416.2, U402.1 (A0), U402.2 (A1), U402.3 (A2), U402.4 (A3), U404.2 (A1), U404.3 (A2)
- net B0: now also C401.1, R403.1; no longer S401.1
- net B1: now also C402.1, R404.1; no longer S402.1
- net B10: now also C411.1, R437.1; no longer S411.1
- net B11: now also C412.1, R438.1; no longer S412.1
- net B12: now also C413.1, R451.1; no longer S413.1
- net B13: now also C414.1, R452.1; no longer S414.1
- net B14: now also C415.1, R453.1; no longer S415.1
- net B15: now also C416.1, R454.1; no longer S416.1
- net B2: now also C403.1, R405.1; no longer S403.1
- net B3: now also C404.1, R406.1; no longer S404.1
- net B4: now also C405.1, R419.1; no longer S405.1
- net B5: now also C406.1, R420.1; no longer S406.1
- net B6: now also C407.1, R421.1; no longer S407.1
- net B7: now also C408.1, R422.1; no longer S408.1
- net B8: now also C409.1, R435.1; no longer S409.1
- net B9: now also C410.1, R436.1; no longer S410.1
- net GND: now also C401.2, C402.2, C403.2, S401.2, S402.2, S403.2, S404.2, S405.2, S406.2, S407.2, S408.2, S409.2, S410.2, S411.2, S412.2, S413.2, S414.2, S415.2, S416.2, SW401.C (Common), SW402.C (Common), SW403.C (Common), U402.1 (A0), U402.2 (A1), U402.3 (A2), U402.4 (A3), U404.2 (A1), U404.3 (A2), C404.2, C405.2, C406.2, C407.2, C408.2, C409.2, C410.2, C411.2, C412.2, C413.2, C414.2, C415.2, C416.2, R401.1, R402.1; no longer SW401.MP, SW402.MP, SW403.MP
- net at U403.25 (GPA4): no longer U401.13 (SDA)
- net at U403.26 (GPA5): no longer U401.12 (SCK)
- net at U403.27 (GPA6): no longer U401.19 (INTB)
- net at U403.28 (GPA7): no longer U401.20 (INTA)
- net at U402.23 (~{OE}): now also R401.2
- net at U404.23 (~{OE}): now also R402.2
- net INTA_Boutons renamed INTB_1
- net INTB_Boutons renamed INTA_1
- net SCK Expandeur_Boutons renamed I2C_SCL
- net I2C_SCL: now also U401.12 (SCK)
- net SCL_0_3_11_8 renamed I2C_SDA
- net I2C_SDA: now also U401.13 (SDA)
- new net: R437.2, R441.2, S411.1
- new net: R406.2, R410.2, S404.1
- new net: R436.2, R440.2, S410.1
- new net: R404.2, R408.2, S402.1
- new net: R454.2, R458.2, S416.1
- new net: R403.2, R407.2, S401.1
- new net: R420.2, R424.2, S406.1
- new net: R453.2, R457.2, S415.1
- new net: R435.2, R439.2, S409.1
- new net: R422.2, R426.2, S408.1
- new net: R438.2, R442.2, S412.1
- new net: R451.2, R455.2, S413.1
- new net: R452.2, R456.2, S414.1
- new net: R419.2, R423.2, S405.1
- new net: R421.2, R425.2, S407.1
- new net: R405.2, R409.2, S403.1
- new net INTA_2: U401.20 (INTA)
- new net INTB_2: U401.19 (INTB)
- no-connect marks 16 -> 23
Other:
- moved on the sheet: U401, U402, U403, U404
