File: Hardware/Sequencer/GPIO_Expandeur.kicad_sch (KiCad schematic)
At the start: 105 parts, among them SW401 SW_SP4T_NR01104, SW402 SW_SP4T_NR01104, SW403 SW_SP4T_NR01104, U401 MCP23017_SP, U402 PCA9635, U403 MCP23017_SP, U404 PCA9635

Commit message: PCB TERMINE (sauf erreurs bizarres et optimisation)
Connections:
- net B10: now also U401.6 (GPB5); no longer U401.23 (GPA2)
- net B10_B: now also U404.16 (LED9); no longer U404.17 (LED10)
- net B10_R: now also U404.15 (LED8); no longer U404.18 (LED11)
- net B11: now also U401.8 (GPB7); no longer U401.24 (GPA3)
- net B11_B: now also U404.18 (LED11); no longer U404.15 (LED8)
- net B11_R: now also U404.17 (LED10); no longer U404.16 (LED9)
- net B12: now also U401.23 (GPA2); no longer U401.25 (GPA4)
- net B13: now also U401.24 (GPA3); no longer U401.26 (GPA5)
- net B14: now also U401.25 (GPA4); no longer U401.27 (GPA6)
- net B14_B: now also U402.7 (LED1); no longer U402.17 (LED10)
- net B14_R: now also U402.6 (LED0); no longer U402.18 (LED11)
- net B15: now also U401.27 (GPA6); no longer U401.28 (GPA7)
- net B15_B: now also U402.11 (LED5); no longer U402.15 (LED8)
- net B15_R: now also U402.10 (LED4); no longer U402.16 (LED9)
- net B2_B: now also U404.21 (LED14); no longer U404.11 (LED5)
- net B2_R: now also U404.22 (LED15); no longer U404.10 (LED4)
- net B3: now also U401.7 (GPB6); no longer U401.4 (GPB3)
- net B3_B: now also U404.20 (LED13); no longer U404.13 (LED7)
- net B3_R: now also U404.19 (LED12); no longer U404.12 (LED6)
- net B4: now also U401.22 (GPA1); no longer U401.5 (GPB4)
- net B4_B: now also U402.16 (LED9); no longer U402.7 (LED1)
- net B4_R: now also U402.15 (LED8); no longer U402.6 (LED0)
- net B5: now also U401.21 (GPA0); no longer U401.6 (GPB5)
- net B5_B: now also U402.18 (LED11); no longer U402.9 (LED3)
- net B5_R: now also U402.17 (LED10); no longer U402.8 (LED2)
- net B6: now also U401.26 (GPA5); no longer U401.7 (GPB6)
- net B6_B: now also U402.9 (LED3); no longer U402.11 (LED5)
- net B6_R: now also U402.8 (LED2); no longer U402.10 (LED4)
- net B7: now also U401.28 (GPA7); no longer U401.8 (GPB7)
- net B8: now also U401.4 (GPB3); no longer U401.21 (GPA0)
- net B8_B: now also U404.11 (LED5); no longer U404.21 (LED14)
- net B8_R: now also U404.10 (LED4); no longer U404.22 (LED15)
- net B9: now also U401.5 (GPB4); no longer U401.22 (GPA1)
- net B9_B: now also U404.13 (LED7); no longer U404.19 (LED12)
- net B9_R: now also U404.12 (LED6); no longer U404.20 (LED13)
Changed lines of the file:
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@@
 	)
 	(label "B5_B"
-		(at 82.55 234.95 0)
+		(at 82.55 255.27 0)
 		(fields_autoplaced yes)
 		(effects
@@
 	)
 	(label "B11"
-		(at 95.25 142.24 0)
+		(at 95.25 129.54 0)
 		(fields_autoplaced yes)
 		(effects
@@
 	)
 	(label "B15"
-		(at 95.25 152.4 0)
+		(at 95.25 149.86 0)
 		(fields_autoplaced yes)
 		(effects
@@
 	)
 	(label "B9"
-		(at 95.25 137.16 0)
+		(at 95.25 121.92 0)
 		(fields_autoplaced yes)
 		(effects
@@
 	)
 	(label "B2_R"
-		(at 119.38 181.61 0)
+		(at 119.38 209.55 0)
 		(fields_autoplaced yes)
 		(effects
@@
 	)
 	(label "B5_R"
-		(at 82.55 232.41 0)
+		(at 82.55 252.73 0)
 		(fields_autoplaced yes)
 		(effects
@@
 	)
 	(label "B7"
-		(at 95.25 129.54 0)
+		(at 95.25 152.4 0)
 		(fields_autoplaced yes)
 		(effects
@@
 	)
 	(label "B15_R"
-		(at 82.55 250.19 0)
+		(at 82.55 237.49 0)
 		(fields_autoplaced yes)
 		(effects
@@
 	)
 	(label "B5"
-		(at 95.25 124.46 0)
+		(at 95.25 134.62 0)
 		(fields_autoplaced yes)
 		(effects
@@
 	)
 	(label "B9_R"
-		(at 119.38 204.47 0)
+		(at 119.38 186.69 0)
 		(fields_autoplaced yes)
 		(effects
@@
 	)
 	(label "B6"
-		(at 95.25 127 0)
+		(at 95.25 147.32 0)
 		(fields_autoplaced yes)
 		(effects
@@
 	)
 	(label "B14_B"
-		(at 82.55 252.73 0)
+		(at 82.55 229.87 0)
 		(fields_autoplaced yes)
 		(effects
@@
 	)
 	(label "B10_R"
-		(at 119.38 199.39 0)
+		(at 119.38 191.77 0)
 		(fields_autoplaced yes)
 		(effects
@@
 	)
 	(label "B8"
-		(at 95.25 134.62 0)
+		(at 95.25 119.38 0)
 		(fields_autoplaced yes)
 		(effects
@@
 	)
 	(label "B11_B"
-		(at 119.38 191.77 0)
+		(at 119.38 199.39 0)
 		(fields_autoplaced yes)
 		(effects
@@
 	)
 	(label "B12"
-		(at 95.25 144.78 0)
+		(at 95.25 139.7 0)
 		(fields_autoplaced yes)
 		(effects
@@
 	)
 	(label "B14_R"
-		(at 82.55 255.27 0)
+		(at 82.55 227.33 0)
 		(fields_autoplaced yes)
 		(effects
@@
 	)
 	(label "B13"
-		(at 95.25 147.32 0)
+		(at 95.25 142.24 0)
 		(fields_autoplaced yes)
 		(effects
@@
 	)
 	(label "B14"
-		(at 95.25 149.86 0)
+		(at 95.25 144.78 0)
 		(fields_autoplaced yes)
 		(effects
@@
 	)
 	(label "B8_B"
-		(at 119.38 207.01 0)
+		(at 119.38 184.15 0)
 		(fields_autoplaced yes)
 		(effects
@@
 	)
 	(label "B6_R"
-		(at 82.55 237.49 0)
+		(at 82.55 232.41 0)
 		(fields_autoplaced yes)
 		(effects
@@
 	)
 	(label "B10_B"
-		(at 119.38 196.85 0)
+		(at 119.38 194.31 0)
 		(fields_autoplaced yes)
 		(effects
@@
 	)
 	(label "B4"
-		(at 95.25 121.92 0)
+		(at 95.25 137.16 0)
 		(fields_autoplaced yes)
 		(effects
@@
 	)
 	(label "B2_B"
-		(at 119.38 184.15 0)
+		(at 119.38 207.01 0)
 		(fields_autoplaced yes)
 		(effects
@@
 	)
 	(label "B3"
-		(at 95.25 119.38 0)
+		(at 95.25 127 0)
 		(fields_autoplaced yes)
 		(effects
@@
 	)
 	(label "B8_R"
-		(at 119.38 209.55 0)
+		(at 119.38 181.61 0)
 		(fields_autoplaced yes)
 		(effects
@@
 	)
 	(label "B3_B"
-		(at 119.38 189.23 0)
+		(at 119.38 204.47 0)
 		(fields_autoplaced yes)
 		(effects
@@
 	)
 	(label "B6_B"
-		(at 82.55 240.03 0)
+		(at 82.55 234.95 0)
 		(fields_autoplaced yes)
 		(effects
@@
 	)
 	(label "B10"
-		(at 95.25 139.7 0)
+		(at 95.25 124.46 0)
 		(fields_autoplaced yes)
 		(effects
@@
 	)
 	(label "B11_R"
-		(at 119.38 194.31 0)
+		(at 119.38 196.85 0)
 		(fields_autoplaced yes)
 		(effects
@@
 	)
 	(label "B15_B"
-		(at 82.55 247.65 0)
+		(at 82.55 240.03 0)
 		(fields_autoplaced yes)
 		(effects
@@
 	)
 	(label "B3_R"
-		(at 119.38 186.69 0)
+		(at 119.38 201.93 0)
 		(fields_autoplaced yes)
 		(effects
@@
 	)
 	(label "B4_R"
-		(at 82.55 227.33 0)
+		(at 82.55 247.65 0)
 		(fields_autoplaced yes)
 		(effects
@@
 	)
 	(label "B4_B"
-		(at 82.55 229.87 0)
+		(at 82.55 250.19 0)
 		(fields_autoplaced yes)
 		(effects
@@
 	)
 	(label "B9_B"
-		(at 119.38 201.93 0)
-		(fields_autoplaced yes)
-		(effects
+		(at 119.38 189.23 0)
+		(fields_autoplaced yes)
+		(effects
